Commit message: correcting joints limits creating srdf file Correcting collision geometries of robots

File: irp6_description/robots/irp6pboth.urdf.xacro (robot description, xacro)
@@ -76,10 +76,10 @@
   <origin xyz="0 0 .25" rpy="0 0 0" />
   <axis xyz="0 1 0" />
-  <limit upper="1.209" lower="0" effort="10" velocity=".53" />
+  <limit upper="1.209" lower="0" effort="10" velocity=".02" />
 </joint>
   <joint name="Irp6otmJoint2" type="revolute">
     <origin rpy="0 0 0" xyz="0.0 0.0 0.3"/>
     <axis xyz="0 0 1"/>
-    <limit lower="-2.96705973" upper="2.96705973" effort="10.0" velocity="10.0" />
+    <limit lower="-2.96705973" upper="2.96705973" effort="10.0" velocity="0.1" />
     <parent link="tl_t"/>
     <child link="tl_1"/>
@@ -108,5 +108,5 @@
     <origin rpy="-1.570795 0 0" xyz="0.0 0.0 0.4"/>
     <axis xyz="0 0 1"/>
-    <limit lower="-1.8" upper="-0.872664626" effort="10.0" velocity="10.0" />
+    <limit lower="-1.8" upper="-0.872664626" effort="10.0" velocity="0.1" />
     <parent link="tl_1"/>
     <child link="tl_2"/>
@@ -134,5 +134,5 @@
     <origin rpy="0 0 0.0" xyz="0.455 0.0 0.0"/>
     <axis xyz="0 0 1"/>
-    <limit lower="-0.3" upper="0.5" effort="10.0" velocity="10.0" />
+    <limit lower="-0.3" upper="0.3" effort="10.0" velocity="0.1" />
     <parent link="tl_2"/>
     <child link="tl_3"/>
@@ -151,7 +151,7 @@
     </visual>
     <collision>
-      <origin rpy="0 0 1.57" xyz="0 0.67 0.0"/>
-      <geometry>
-        <mesh filename="package://irp6_description/meshes/link3.stlb" scale="1.0 1.0 1.3" />
+      <origin rpy="0 0 1.57" xyz="0 0.70 0.0"/>
+      <geometry>
+        <mesh filename="package://irp6_description/meshes/link3.stlb" scale="1.05 1.3 1.5" />
       </geometry>
     </collision>
@@ -160,5 +160,5 @@
     <origin rpy="0 0 0" xyz="0.0 0.67 0.0"/>
     <axis xyz="0 0 1"/>
-    <limit lower="-1.57" upper="1.57" effort="10.0" velocity="10.0" />
+    <limit lower="-1.57" upper="1.57" effort="10.0" velocity="0.1" />
     <parent link="tl_3"/>
     <child link="tl_4"/>
@@ -186,5 +186,5 @@
     <origin rpy="-1.570795 0 0" xyz="0.0 0.0 0.0"/>
     <axis xyz="0 0 1"/>
-    <limit lower="-0.5" upper="5.14" effort="10.0" velocity="10.0" />
+    <limit lower="0.5" upper="5.14" effort="10.0" velocity="0.1" />
     <parent link="tl_4"/>
     <child link="tl_5"/>
@@ -205,5 +205,5 @@
       <origin rpy="1.57 0 0.0" xyz="0.0 0.0 0.19"/>
       <geometry>
-        <mesh filename="package://irp6_description/meshes/link5.stlb" />
+        <mesh filename="package://irp6_description/meshes/link5.stlb" scale="2 2 1.1" />
       </geometry>
     </collision>
@@ -212,5 +212,5 @@
     <origin rpy="1.570795 0 0" xyz="0.0 0.0 0.19"/>
     <axis xyz="0 0 1"/>
-    <limit lower="-3.0" upper="2.9" effort="10.0" velocity="10.0" />
+    <limit lower="-2.9" upper="2.8" effort="10.0" velocity="0.1" />
     <parent link="tl_5"/>
     <child link="tl_6"/>
@@ -229,7 +229,7 @@
     </visual>
     <collision>
-      <origin rpy="0.0 0 0.0" xyz="0 0.0 -0.05"/>
-      <geometry>
-        <cylinder radius="0.1" length="0.10" />
+      <origin rpy="0.0 0 0.0" xyz="0 0.0 0.10"/>
+      <geometry>
+        <cylinder radius="0.12" length="0.10" />
       </geometry>
     </collision>
@@ -263,7 +263,7 @@
     </visual>
     <collision>
-      <origin rpy="0.0 0 0.0" xyz="0 0.02 0.0"/>
-      <geometry>
-        <box size="0.05 0.04 0.12" />
+      <origin rpy="0.0 0 0.0" xyz="0 0.02 0.05"/>
+      <geometry>
+        <box size="0.08 0.06 0.18" />
       </geometry>
     </collision>
@@ -282,7 +282,7 @@
     </visual>
     <collision>
-      <origin rpy="0.0 0 0.0" xyz="0 -0.02 0.0"/>
-      <geometry>
-        <box size="0.05 0.04 0.12" />
+      <origin rpy="0.0 0 0.0" xyz="0 -0.02 0.05"/>
+      <geometry>
+        <box size="0.08 0.06 0.18" />
       </geometry>
     </collision>
@@ -335,5 +335,5 @@
     <origin rpy="0 0 0" xyz="0.0 0.0 0.55"/>
     <axis xyz="0 0 1"/>
-    <limit lower="-2.96705973" upper="2.96705973" effort="10.0" velocity="10.0" />
+    <limit lower="-2.96705973" upper="2.96705973" effort="10.0" velocity="0.1" />
     <parent link="pl_base"/>
     <child link="pl_1"/>
@@ -362,5 +362,5 @@
     <origin rpy="-1.570795 0 0" xyz="0.0 0.0 0.4"/>
     <axis xyz="0 0 1"/>
-    <limit lower="-1.8" upper="-0.872664626" effort="10.0" velocity="10.0" />
+    <limit lower="-1.8" upper="-0.872664626" effort="10.0" velocity="0.1" />
     <parent link="pl_1"/>
     <child link="pl_2"/>
@@ -388,5 +388,5 @@
     <origin rpy="0 0 0.0" xyz="0.455 0.0 0.0"/>
     <axis xyz="0 0 1"/>
-    <limit lower="-0.3" upper="0.5" effort="10.0" velocity="10.0" />
+    <limit lower="-0.3" upper="0.3" effort="10.0" velocity="0.1" />
     <parent link="pl_2"/>
     <child link="pl_3"/>
@@ -407,5 +407,5 @@
       <origin rpy="0 0 1.57" xyz="0 0.67 0.0"/>
       <geometry>
-        <mesh filename="package://irp6_description/meshes/link3.stlb" scale="1.0 1.0 1.3" />
+        <mesh filename="package://irp6_description/meshes/link3.stlb" scale="1.05 1.3 1.5" />
       </geometry>
     </collision>
@@ -414,5 +414,5 @@
     <origin rpy="0 0 0" xyz="0.0 0.67 0.0"/>
     <axis xyz="0 0 1"/>
-    <limit lower="-1.57" upper="1.57" effort="10.0" velocity="10.0" />
+    <limit lower="-1.57" upper="1.57" effort="10.0" velocity="0.1" />
     <parent link="pl_3"/>
     <child link="pl_4"/>
@@ -440,5 +440,5 @@
     <origin rpy="-1.570795 0 0" xyz="0.0 0.0 0.0"/>
     <axis xyz="0 0 1"/>
-    <limit lower="-0.5" upper="5.14" effort="10.0" velocity="10.0" />
+    <limit lower="0.5" upper="5.14" effort="10.0" velocity="0.1" />
     <parent link="pl_4"/>
     <child link="pl_5"/>
@@ -459,5 +459,5 @@
       <origin rpy="1.57 0 0.0" xyz="0.0 0.0 0.19"/>
       <geometry>
-        <mesh filename="package://irp6_description/meshes/link5.stlb" />
+        <mesh filename="package://irp6_description/meshes/link5.stlb" scale="2 2 1.1"/>
       </geometry>
     </collision>
@@ -466,5 +466,5 @@
     <origin rpy="1.570795 0 0" xyz="0.0 0.0 0.19"/>
     <axis xyz="0 0 1"/>
-    <limit lower="-3.0" upper="2.9" effort="10.0" velocity="10.0" />
+    <limit lower="-3.0" upper="2.9" effort="10.0" velocity="0.1" />
     <parent link="pl_5"/>
     <child link="pl_6"/>
@@ -483,7 +483,7 @@
     </visual>
     <collision>
-      <origin rpy="0.0 0 0.0" xyz="0 0.0 -0.05"/>
-      <geometry>
-        <cylinder radius="0.1" length="0.10" />
+      <origin rpy="0.0 0 0.0" xyz="0 0.0 0.1"/>
+      <geometry>
+        <cylinder radius="0.12" length="0.10" />
       </geometry>
     </collision>
@@ -517,7 +517,7 @@
     </visual>
     <collision>
-      <origin rpy="0.0 0 0.0" xyz="0 0.02 0.0"/>
-      <geometry>
-        <box size="0.05 0.04 0.12" />
+      <origin rpy="0.0 0 0.0" xyz="0 0.02 0.05"/>
+      <geometry>
+        <box size="0.08 0.06 0.18" />
       </geometry>
     </collision>
@@ -536,7 +536,7 @@
     </visual>
     <collision>
-      <origin rpy="0.0 0 0.0" xyz="0 -0.02 0.0"/>
-      <geometry>
-        <box size="0.05 0.04 0.12" />
+      <origin rpy="0.0 0 0.0" xyz="0 -0.02 0.05"/>
+      <geometry>
+        <box size="0.08 0.06 0.18" />
       </geometry>
     </collision>

Commit message: correct collision geometry

File: irp6_description/robots/irp6pboth.urdf.xacro (robot description, xacro)
@@ -134,5 +134,5 @@
     <origin rpy="0 0 0.0" xyz="0.455 0.0 0.0"/>
     <axis xyz="0 0 1"/>
-    <limit lower="-0.3" upper="0.3" effort="10.0" velocity="0.1" />
+    <limit lower="-0.5" upper="0.3" effort="10.0" velocity="0.1" />
     <parent link="tl_2"/>
     <child link="tl_3"/>
@@ -205,5 +205,5 @@
       <origin rpy="1.57 0 0.0" xyz="0.0 0.0 0.19"/>
       <geometry>
-        <mesh filename="package://irp6_description/meshes/link5.stlb" scale="2 2 1.1" />
+        <mesh filename="package://irp6_description/meshes/link5.stlb" scale="2.2 2.2 1.1" />
       </geometry>
     </collision>
@@ -212,5 +212,5 @@
     <origin rpy="1.570795 0 0" xyz="0.0 0.0 0.19"/>
     <axis xyz="0 0 1"/>
-    <limit lower="-2.9" upper="2.8" effort="10.0" velocity="0.1" />
+    <limit lower="-2.8" upper="2.8" effort="10.0" velocity="0.1" />
     <parent link="tl_5"/>
     <child link="tl_6"/>
@@ -263,7 +263,7 @@
     </visual>
     <collision>
-      <origin rpy="0.0 0 0.0" xyz="0 0.02 0.05"/>
-      <geometry>
-        <box size="0.08 0.06 0.18" />
+      <origin rpy="0.0 0 0.0" xyz="0 0.02 0.0"/>
+      <geometry>
+        <box size="0.08 0.06 0.20" />
       </geometry>
     </collision>
@@ -282,7 +282,7 @@
     </visual>
     <collision>
-      <origin rpy="0.0 0 0.0" xyz="0 -0.02 0.05"/>
-      <geometry>
-        <box size="0.08 0.06 0.18" />
+      <origin rpy="0.0 0 0.0" xyz="0 -0.02 0.0"/>
+      <geometry>
+        <box size="0.08 0.06 0.20" />
       </geometry>
     </collision>
@@ -459,5 +459,5 @@
       <origin rpy="1.57 0 0.0" xyz="0.0 0.0 0.19"/>
       <geometry>
-        <mesh filename="package://irp6_description/meshes/link5.stlb" scale="2 2 1.1"/>
+        <mesh filename="package://irp6_description/meshes/link5.stlb" scale="2.2 2.2 1.1"/>
       </geometry>
     </collision>
@@ -517,7 +517,7 @@
     </visual>
     <collision>
-      <origin rpy="0.0 0 0.0" xyz="0 0.02 0.05"/>
-      <geometry>
-        <box size="0.08 0.06 0.18" />
+      <origin rpy="0.0 0 0.0" xyz="0 0.02 0.0"/>
+      <geometry>
+        <box size="0.08 0.06 0.20" />
       </geometry>
     </collision>
@@ -536,7 +536,7 @@
     </visual>
     <collision>
-      <origin rpy="0.0 0 0.0" xyz="0 -0.02 0.05"/>
-      <geometry>
-        <box size="0.08 0.06 0.18" />
+      <origin rpy="0.0 0 0.0" xyz="0 -0.02 0.0"/>
+      <geometry>
+        <box size="0.08 0.06 0.20" />
       </geometry>
     </collision>

Commit message: correct irp6 collision model

File: irp6_description/robots/irp6pboth.urdf.xacro (robot description, xacro)
@@ -265,5 +265,5 @@
       <origin rpy="0.0 0 0.0" xyz="0 0.02 0.0"/>
       <geometry>
-        <box size="0.08 0.06 0.20" />
+        <box size="0.08 0.05 0.20" />
       </geometry>
     </collision>
@@ -284,5 +284,5 @@
       <origin rpy="0.0 0 0.0" xyz="0 -0.02 0.0"/>
       <geometry>
-        <box size="0.08 0.06 0.20" />
+        <box size="0.08 0.05 0.20" />
       </geometry>
     </collision>
@@ -483,7 +483,7 @@
     </visual>
     <collision>
-      <origin rpy="0.0 0 0.0" xyz="0 0.0 0.1"/>
-      <geometry>
-        <cylinder radius="0.12" length="0.10" />
+      <origin rpy="1.570795 0.0 0.0" xyz="0 0.0 0.0"/>
+      <geometry>
+        <mesh filename="package://irp6_description/meshes/link62.3ds" scale = "0.15 0.15 0.15" />
       </geometry>
     </collision>
@@ -519,5 +519,5 @@
       <origin rpy="0.0 0 0.0" xyz="0 0.02 0.0"/>
       <geometry>
-        <box size="0.08 0.06 0.20" />
+        <box size="0.03 0.01 0.20" />
       </geometry>
     </collision>
@@ -538,5 +538,5 @@
       <origin rpy="0.0 0 0.0" xyz="0 -0.02 0.0"/>
       <geometry>
-        <box size="0.08 0.06 0.20" />
+        <box size="0.03 0.01 0.20" />
       </geometry>
     </collision>

Commit message: magiczna liczba poprawa modeli

File: irp6_description/robots/irp6pboth.urdf.xacro (robot description, xacro)
@@ -108,5 +108,5 @@
     <origin rpy="-1.570795 0 0" xyz="0.0 0.0 0.4"/>
     <axis xyz="0 0 1"/>
-    <limit lower="-1.8" upper="-0.872664626" effort="10.0" velocity="0.1" />
+    <limit lower="-1.6" upper="-0.272664626" effort="10.0" velocity="0.1" />
     <parent link="tl_1"/>
     <child link="tl_2"/>
@@ -229,7 +229,7 @@
     </visual>
     <collision>
-      <origin rpy="0.0 0 0.0" xyz="0 0.0 0.10"/>
-      <geometry>
-        <cylinder radius="0.12" length="0.10" />
+     <origin rpy="1.570795 0.0 0.0" xyz="0 0.0 0.0"/>
+      <geometry>
+        <mesh filename="package://irp6_description/meshes/link62.3ds" scale = "0.15 0.15 0.15" />
       </geometry>
     </collision>
@@ -240,5 +240,5 @@
     <child link="tl_g1"/>
     <axis xyz="0 1 0" />
-    <limit upper="0.1" lower="0" effort="10" velocity=".53" />
+    <limit upper="0.1" lower="0.05" effort="10" velocity=".005" />
   </joint>
   <joint name="Irp6ottfgJoint1a" type="prismatic">
@@ -247,5 +247,5 @@
     <child link="tl_g2"/>
     <axis xyz="0 -1 0" />
-    <limit upper="0.1" lower="0" effort="10" velocity=".53" />
+    <limit upper="0.1" lower="0.05" effort="10" velocity=".005" />
     <mimic joint="Irp6ottfgJoint1" />
   </joint>
@@ -257,5 +257,5 @@
     </inertial>
     <visual>
-      <origin rpy="0 0 0.0" xyz="0 0.02 0.0"/>
+      <origin rpy="0 0 0.0" xyz="0 0.00 0.0"/>
       <geometry>
          <box size="0.05 0.04 0.12" />
@@ -263,7 +263,7 @@
     </visual>
     <collision>
-      <origin rpy="0.0 0 0.0" xyz="0 0.02 0.0"/>
-      <geometry>
-        <box size="0.08 0.05 0.20" />
+      <origin rpy="0.0 0 0.0" xyz="0 0.00 0.0"/>
+      <geometry>
+        <box size="0.03 0.01 0.18" />
       </geometry>
     </collision>
@@ -276,5 +276,5 @@
     </inertial>
     <visual>
-      <origin rpy="0 0 0.0" xyz="0 -0.02 0.0"/>
+      <origin rpy="0 0 0.0" xyz="0 -0.00 0.0"/>
       <geometry>
          <box size="0.05 0.04 0.12" />
@@ -282,7 +282,7 @@
     </visual>
     <collision>
-      <origin rpy="0.0 0 0.0" xyz="0 -0.02 0.0"/>
-      <geometry>
-        <box size="0.08 0.05 0.20" />
+      <origin rpy="0.0 0 0.0" xyz="0 -0.00 0.0"/>
+      <geometry>
+        <box size="0.03 0.01 0.18" />
       </geometry>
     </collision>
@@ -362,5 +362,5 @@
     <origin rpy="-1.570795 0 0" xyz="0.0 0.0 0.4"/>
     <axis xyz="0 0 1"/>
-    <limit lower="-1.8" upper="-0.872664626" effort="10.0" velocity="0.1" />
+    <limit lower="-1.6" upper="-0.272664626" effort="10.0" velocity="0.1" />
     <parent link="pl_1"/>
     <child link="pl_2"/>
@@ -388,5 +388,5 @@
     <origin rpy="0 0 0.0" xyz="0.455 0.0 0.0"/>
     <axis xyz="0 0 1"/>
-    <limit lower="-0.3" upper="0.3" effort="10.0" velocity="0.1" />
+    <limit lower="-0.2" upper="0.2" effort="10.0" velocity="0.1" />
     <parent link="pl_2"/>
     <child link="pl_3"/>
@@ -494,5 +494,5 @@
     <child link="pl_g1"/>
     <axis xyz="0 1 0" />
-    <limit upper="0.1" lower="0" effort="10" velocity=".53" />
+    <limit upper="0.1" lower="0.00" effort="10" velocity=".005" />
   </joint>
   <joint name="Irp6ptfgJoint1a" type="prismatic">
@@ -501,5 +501,5 @@
     <child link="pl_g2"/>
     <axis xyz="0 -1 0" />
-    <limit upper="0.1" lower="0" effort="10" velocity=".53" />
+    <limit upper="0.1" lower="0.00" effort="10" velocity=".005" />
     <mimic joint="Irp6ptfgJoint1" />
   </joint>
@@ -511,5 +511,5 @@
     </inertial>
     <visual>
-      <origin rpy="0 0 0.0" xyz="0 0.02 0.0"/>
+      <origin rpy="0 0 0.0" xyz="0 0.00 0.0"/>
       <geometry>
          <box size="0.05 0.04 0.12" />
@@ -517,5 +517,5 @@
     </visual>
     <collision>
-      <origin rpy="0.0 0 0.0" xyz="0 0.02 0.0"/>
+      <origin rpy="0.0 0 0.0" xyz="0 0.00 0.0"/>
       <geometry>
         <box size="0.03 0.01 0.20" />
@@ -530,5 +530,5 @@
     </inertial>
     <visual>
-      <origin rpy="0 0 0.0" xyz="0 -0.02 0.0"/>
+      <origin rpy="0 0 0.0" xyz="0 -0.00 0.0"/>
       <geometry>
          <box size="0.05 0.04 0.12" />
@@ -536,7 +536,7 @@
     </visual>
     <collision>
-      <origin rpy="0.0 0 0.0" xyz="0 -0.02 0.0"/>
-      <geometry>
-        <box size="0.03 0.01 0.20" />
+      <origin rpy="0.0 0 0.0" xyz="0 -0.00 0.0"/>
+      <geometry>
+        <box size="0.03 0.01 0.18" />
       </geometry>
     </collision>

Commit message: correct front position correct joint limits

File: irp6_description/robots/irp6pboth.urdf.xacro (robot description, xacro)
@@ -466,5 +466,5 @@
     <origin rpy="1.570795 0 0" xyz="0.0 0.0 0.19"/>
     <axis xyz="0 0 1"/>
-    <limit lower="-3.0" upper="2.9" effort="10.0" velocity="0.1" />
+    <limit lower="-2.88" upper="2.88" effort="10.0" velocity="0.1" />
     <parent link="pl_5"/>
     <child link="pl_6"/>

Commit message: correct joints limits

File: irp6_description/robots/irp6pboth.urdf.xacro (robot description, xacro)
@@ -81,5 +81,5 @@
     <origin rpy="0 0 0" xyz="0.0 0.0 0.3"/>
     <axis xyz="0 0 1"/>
-    <limit lower="-2.96705973" upper="2.96705973" effort="10.0" velocity="0.1" />
+    <limit lower="-2.96705973" upper="2.96705973" effort="10.0" velocity="0.5" />
     <parent link="tl_t"/>
     <child link="tl_1"/>
@@ -108,5 +108,5 @@
     <origin rpy="-1.570795 0 0" xyz="0.0 0.0 0.4"/>
     <axis xyz="0 0 1"/>
-    <limit lower="-1.6" upper="-0.272664626" effort="10.0" velocity="0.1" />
+    <limit lower="-1.6" upper="-1.02664626" effort="10.0" velocity="0.5" />
     <parent link="tl_1"/>
     <child link="tl_2"/>
@@ -134,5 +134,5 @@
     <origin rpy="0 0 0.0" xyz="0.455 0.0 0.0"/>
     <axis xyz="0 0 1"/>
-    <limit lower="-0.5" upper="0.3" effort="10.0" velocity="0.1" />
+    <limit lower="-0.3" upper="0.3" effort="10.0" velocity="0.5" />
     <parent link="tl_2"/>
     <child link="tl_3"/>
@@ -160,5 +160,5 @@
     <origin rpy="0 0 0" xyz="0.0 0.67 0.0"/>
     <axis xyz="0 0 1"/>
-    <limit lower="-1.57" upper="1.57" effort="10.0" velocity="0.1" />
+    <limit lower="-1.57" upper="1.57" effort="10.0" velocity="0.5" />
     <parent link="tl_3"/>
     <child link="tl_4"/>
@@ -186,5 +186,5 @@
     <origin rpy="-1.570795 0 0" xyz="0.0 0.0 0.0"/>
     <axis xyz="0 0 1"/>
-    <limit lower="0.5" upper="5.14" effort="10.0" velocity="0.1" />
+    <limit lower="0.5" upper="5.14" effort="10.0" velocity="0.5" />
     <parent link="tl_4"/>
     <child link="tl_5"/>
@@ -212,5 +212,5 @@
     <origin rpy="1.570795 0 0" xyz="0.0 0.0 0.19"/>
     <axis xyz="0 0 1"/>
-    <limit lower="-2.8" upper="2.8" effort="10.0" velocity="0.1" />
+    <limit lower="-2.8" upper="2.8" effort="10.0" velocity="0.5" />
     <parent link="tl_5"/>
     <child link="tl_6"/>
@@ -335,5 +335,5 @@
     <origin rpy="0 0 0" xyz="0.0 0.0 0.55"/>
     <axis xyz="0 0 1"/>
-    <limit lower="-2.96705973" upper="2.96705973" effort="10.0" velocity="0.1" />
+    <limit lower="-2.96705973" upper="2.96705973" effort="10.0" velocity="0.6" />
     <parent link="pl_base"/>
     <child link="pl_1"/>
@@ -362,5 +362,5 @@
     <origin rpy="-1.570795 0 0" xyz="0.0 0.0 0.4"/>
     <axis xyz="0 0 1"/>
-    <limit lower="-1.6" upper="-0.272664626" effort="10.0" velocity="0.1" />
+    <limit lower="-1.6" upper="-0.272664626" effort="10.0" velocity="0.5" />
     <parent link="pl_1"/>
     <child link="pl_2"/>
@@ -388,5 +388,5 @@
     <origin rpy="0 0 0.0" xyz="0.455 0.0 0.0"/>
     <axis xyz="0 0 1"/>
-    <limit lower="-0.2" upper="0.2" effort="10.0" velocity="0.1" />
+    <limit lower="-0.2" upper="0.2" effort="10.0" velocity="0.5" />
     <parent link="pl_2"/>
     <child link="pl_3"/>
@@ -414,5 +414,5 @@
     <origin rpy="0 0 0" xyz="0.0 0.67 0.0"/>
     <axis xyz="0 0 1"/>
-    <limit lower="-1.57" upper="1.57" effort="10.0" velocity="0.1" />
+    <limit lower="-1.57" upper="1.57" effort="10.0" velocity="0.5" />
     <parent link="pl_3"/>
     <child link="pl_4"/>
@@ -440,5 +440,5 @@
     <origin rpy="-1.570795 0 0" xyz="0.0 0.0 0.0"/>
     <axis xyz="0 0 1"/>
-    <limit lower="0.5" upper="5.14" effort="10.0" velocity="0.1" />
+    <limit lower="0.5" upper="5.14" effort="10.0" velocity="0.5" />
     <parent link="pl_4"/>
     <child link="pl_5"/>
@@ -466,5 +466,5 @@
     <origin rpy="1.570795 0 0" xyz="0.0 0.0 0.19"/>
     <axis xyz="0 0 1"/>
-    <limit lower="-2.88" upper="2.88" effort="10.0" velocity="0.1" />
+    <limit lower="-2.88" upper="2.88" effort="10.0" velocity="0.5" />
     <parent link="pl_5"/>
     <child link="pl_6"/>
